File: Schematic/Ram_Tester.kicad_sch (KiCad schematic)
At the start: 19 parts, among them J1 Conn_01x02_Pin, J2 ICSP, SW1 SW_DIP_x03, U1 ATmega328-P, U2 RAM / ZIF, U3 ZIP Socket, U4 DIP Socket, Y1 Crystal

Commit message: v1.0 of PCB
Parts:
- added C5: 10uF, Capacitor_SMD:C_1206_3216Metric, symbol Device:C_Polarized
- added C6, C7: 100nF, Capacitor_SMD:C_0805_2012Metric, symbol Device:C
- added Q1, Q2: IRLML6402, Package_TO_SOT_SMD:SOT-23, symbol Transistor_FET:IRLML6402
- added R7, R8: 47, Resistor_SMD:R_0603_1608Metric, symbol Device:R
- added RN1, RN2, RN3, RN4: 47, Resistor_SMD:R_Array_Concave_4x0603, symbol Device:R_Pack04
- added SW2: SW_Push, Button_Switch_SMD:TLZWLA_Button, symbol Switch:SW_MEC_5E
- J1: footprint Connector_PinHeader_2.54mm:PinHeader_1x02_P2.54mm_Vertical -> Connector_USB:MicroUSB PowerOnly
- U1: footprint Socket:DIP_Socket-28_W6.9_W7.62_W10.16_W12.7_W13.5_3M_228-4817-00-0602J -> Package_DIP:DIP-28_W7.62mm
Connections:
- net 5V: now also C5.1, C7.2, Q1.3 (D), Q2.3 (D)
- net GND: now also C5.2, C6.2, C7.1, SW2.1, SW2.2
- net at J2.1 (Pin_1), U1.18 (PB4): now also Q1.1 (G), R7.1; no longer R1.1, U2.15 (A8)
- net at D1.3 (K): now also R1.1; no longer R1.2
- net at R3.2, SW1.6, U1.28 (PC5)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: now also C6.1
- net at J2.3 (Pin_3), U1.19 (PB5): now also Q2.1 (G); no longer R6.1
- net at J2.4 (Pin_4), U2.3 (WE): now also RN1.1 (R1.1); no longer U1.17 (PB3)
- net at J2.5 (Pin_5), R2.2, U1.1 (~{RESET}/PC6): now also SW2.3 (K), SW2.4 (A)
- net at R5.2, SW1.4, U2.8 (A2): now also RN3.3 (R3.1); no longer U1.4 (PD2)
- net at R4.2, SW1.5, U2.9 (A3): now also RN3.4 (R4.1); no longer U1.5 (PD3)
- net at U2.1 (I/O1): now also RN4.4 (R4.1); no longer U1.23 (PC0)
- net at U2.11 (A4): now also RN2.4 (R4.1); no longer U1.6 (PD4)
- net at U2.12 (A5): now also RN2.3 (R3.1); no longer U1.11 (PD5)
- net at U2.13 (A6): now also RN2.2 (R2.1); no longer U1.12 (PD6)
- net at U2.14 (A7): now also RN2.1 (R1.1); no longer U1.13 (PD7)
- net at U2.16 (OE): now also RN1.2 (R2.1); no longer U1.16 (PB2)
- net at U2.17 (CAS): now also RN1.4 (R4.1); no longer U1.14 (PB0)
- net at U2.18 (I/O3): now also RN4.2 (R2.1); no longer U1.25 (PC2)
- net at U2.19 (I/O4): now also RN4.1 (R1.1); no longer U1.26 (PC3)
- net at U2.2 (I/O2): now also RN4.3 (R3.1); no longer U1.24 (PC1)
- net at U2.4 (RAS): now also RN1.3 (R3.1); no longer U1.15 (PB1)
- net at U1.27 (PC4): now also R8.1; no longer U2.5 (N/C)
- net at U2.6 (A0): now also RN3.1 (R1.1); no longer U1.2 (PD0)
- net at U2.7 (A1): now also RN3.2 (R2.1); no longer U1.3 (PD1)
- new net: RN4.5 (R4.2), U1.23 (PC0)
- new net: RN4.6 (R3.2), U1.24 (PC1)
- new net: RN4.7 (R2.2), U1.25 (PC2)
- new net: RN4.8 (R1.2), U1.26 (PC3)
- new net: RN3.5 (R4.2), U1.5 (PD3)
- new net: RN3.6 (R3.2), U1.4 (PD2)
- new net: RN3.7 (R2.2), U1.3 (PD1)
- new net: RN3.8 (R1.2), U1.2 (PD0)
- new net: R8.2, U2.5 (N/C)
- new net: Q1.2 (S), R1.2
- new net: Q2.2 (S), R6.1
- new net: R7.2, U2.15 (A8)
- new net: RN2.5 (R4.2), U1.6 (PD4)
- new net: RN2.6 (R3.2), U1.11 (PD5)
- new net: RN2.7 (R2.2), U1.12 (PD6)
- new net: RN2.8 (R1.2), U1.13 (PD7)
- new net: RN1.5 (R4.2), U1.14 (PB0)
- new net: RN1.6 (R3.2), U1.15 (PB1)
- new net: RN1.7 (R2.2), U1.16 (PB2)
- new net: RN1.8 (R1.2), U1.17 (PB3)
Other:
- moved on the sheet: D1, J1, R1, R6
