File: Schematic/TH/Ram_Tester.kicad_sch (KiCad schematic)
At the start: 42 parts, among them J1 Conn_01x02_Pin, J2 ICSP, Q1 2N7000, Q2 2N7000, SW1 SW_DIP_x03, SW2 SW_Push, U1 ATmega328-P, U2 RAM / ZIF, U3 ZIP Socket, Y1 16MHz

Commit message: v1.1 - minor fix
Parts:
- C5: footprint Capacitor_THT:C_Disc_D4.3mm_W1.9mm_P5.00mm -> Capacitor_THT:CP_Radial_D4.0mm_P2.00mm
- Y1: value 16MHz -> Crystal
Changed lines of the file:
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@@
 			)
 		)
-		(property "Value" "16MHz"
+		(property "Value" "Crystal"
 			(at 112.522 91.186 0)
 			(effects
@@
 			)
 		)
-		(property "Footprint" "Capacitor_THT:C_Disc_D4.3mm_W1.9mm_P5.00mm"
+		(property "Footprint" "Capacitor_THT:CP_Radial_D4.0mm_P2.00mm"
 			(at 44.1452 142.24 0)
 			(effects
