File: Schematic/TH/Ram_Tester.kicad_pcb (KiCad board)
At the start: 2 copper layers, 63.3 x 57.2 mm, 43 parts, among them J1 Conn_01x02_Pin, J2 ICSP, Q1 2N7000, Q2 2N7000, SW1 SW_DIP_x03, SW2 SW_Push, U1 ATmega328-P, U2 RAM / ZIF, U3 ZIP Socket, Y1 Crystal

Commit message: Add files via upload
Parts:
- SW2: footprint Button_Switch_THT:SW_TH_Tactile_Omron_B3F-10xx -> Button_Switch_THT:SW_PUSH_6mm_H5mm
- renumbered Display1 to Display
Changed lines of the file:
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@@
 		(tags "CP Radial series Radial pin pitch 2.00mm  diameter 4mm Electrolytic Capacitor")
 		(property "Reference" "C5"
-			(at 4.2606 -0.635 180)
+			(at 2.8626 3.13 180)
 			(layer "F.SilkS")
 			(effects
@@
 		(descr "Through hole straight pin header, 1x04, 2.54mm pitch, single row")
 		(tags "Through hole pin header THT 1x04 2.54mm single row")
-		(property "Reference" "Display1"
-			(at 2.667 3.429 0)
+		(property "Reference" "Display"
+			(at -2.57 3.53 0)
 			(layer "F.SilkS")
 			(effects
@@
 		(sheetname "Root")
 		(sheetfile "Ram_Tester.kicad_sch")
-		(attr through_hole)
+		(attr through_hole dnp)
 		(fp_line
 			(start -1.33 -1.33)
@@
 		(tags "THT DIP DIL PDIP 2.54mm 7.62mm 300mil")
 		(property "Reference" "U1"
-			(at 3.797 -2.286 0)
+			(at 0.09 -2.24 0)
 			(layer "F.SilkS")
 			(effects
@@
 		(tags "DIP Switch SPST Slide 7.62mm 300mil")
 		(property "Reference" "SW1"
-			(at 9.97 -1.12 180)
+			(at 4.42 9.46 180)
 			(layer "F.SilkS")
 			(effects
@@
 		)
 	)
-	(footprint "Button_Switch_THT:SW_TH_Tactile_Omron_B3F-10xx"
+	(footprint "Button_Switch_THT:SW_PUSH_6mm_H5mm"
 		(layer "F.Cu")
 		(at 101.17 76.85 180)
-		(descr "SW_TH_Tactile_Omron_B3F-10xx_https://www.omron.com/ecb/products/pdf/en-b3f.pdf")
-		(tags "Omron B3F-10xx")
+		(descr "tactile push button, 6x6mm e.g. PHAP33xx series, height=5mm")
+		(tags "tact sw push 6mm")
 		(property "Reference" "SW2"
-			(at 3.377 4.409 0)
+			(at 3.25 2.25 180)
 			(layer "F.SilkS")
 			(effects
@@
 		)
 		(property "Value" "SW_Push"
-			(at 3.2 6.5 0)
+			(at 3.75 6.7 180)
 			(layer "F.Fab")
-			(hide yes)
 			(effects
 				(font
@@
 			)
 		)
-		(property "Footprint" "Button_Switch_THT:SW_TH_Tactile_Omron_B3F-10xx"
+		(property "Footprint" "Button_Switch_THT:SW_PUSH_6mm_H5mm"
 			(at 0 0 180)
 			(unlocked yes)
@@
 				(font
 					(size 1.27 1.27)
-					(thickness 0.15)
 				)
 			)
@@
 				(font
 					(size 1.27 1.27)
-					(thickness 0.15)
 				)
 			)
@@
 				(font
 					(size 1.27 1.27)
-					(thickness 0.15)
 				)
 			)
@@
 		(attr through_hole)
 		(fp_line
-			(start 6.37 1.2)
-			(end 6.37 3.4)
+			(start 6.75 3)
+			(end 6.75 1.5)
 			(stroke
 				(width 0.12)
@@
 		)
 		(fp_line
-			(start 1.2 -0.87)
-			(end 5.6 -0.87)
+			(start 5.5 -1)
+			(end 1 -1)
 			(stroke
 				(width 0.12)
@@
 		)
 		(fp_line
-			(start 0.6 5.37)
-			(end 5.8 5.37)
+			(start 1 5.5)
+			(end 5.5 5.5)
 			(stroke
 				(width 0.12)
@@
 		)
 		(fp_line
-			(start 0.13 3.4)
-			(end 0.13 1.2)
+			(start -0.25 1.5)
+			(end -0.25 3)
 			(stroke
 				(width 0.12)
@@
 			(layer "F.SilkS")
 		)
-		(fp_circle
-			(center 3.25 2.25)
-			(end 4.25 3.25)
+		(fp_line
+			(start 8 6)
+			(end 8 5.75)
 			(stroke
-				(width 0.12)
+				(width 0.05)
 				(type solid)
 			)
-			(fill none)
-			(layer "F.SilkS")
+			(layer "F.CrtYd")
 		)
 		(fp_line
-			(start 7.6 5.6)
-			(end 7.6 -1.1)
+			(start 8 -1.25)
+			(end 8 5.75)
 			(stroke
 				(width 0.05)
@@
 		)
 		(fp_line
-			(start -1.1 5.6)
-			(end 7.6 5.6)
+			(start 8 -1.5)
+			(end 8 -1.25)
 			(stroke
 				(width 0.05)
@@
 		)
 		(fp_line
-			(start -1.1 -1.1)
-			(end 7.6 -1.1)
+			(start 7.75 6)
+			(end 8 6)
 			(stroke
 				(width 0.05)
@@
 		)
 		(fp_line
-			(start -1.1 -1.1)
-			(end -1.1 5.6)
+			(start 7.75 6)
+			(end -1.25 6)
 			(stroke
 				(width 0.05)
@@
 		)
 		(fp_line
-			(start 6.25 -0.75)
-			(end 6.25 5.25)
+			(start 7.75 -1.5)
+			(end 8 -1.5)
+			(stroke
+				(width 0.05)
+				(type solid)
+			)
+			(layer "F.CrtYd")
+		)
+		(fp_line
+			(start -1.25 -1.5)
+			(end 7.75 -1.5)
+			(stroke
+				(width 0.05)
+				(type solid)
+			)
+			(layer "F.CrtYd")
+		)
+		(fp_line
+			(start -1.5 6)
+			(end -1.25 6)
+			(stroke
+				(width 0.05)
+				(type solid)
+			)
+			(layer "F.CrtYd")
+		)
+		(fp_line
+			(start -1.5 5.75)
+			(end -1.5 6)
+			(stroke
+				(width 0.05)
+				(type solid)
+			)
+			(layer "F.CrtYd")
+		)
+		(fp_line
+			(start -1.5 5.75)
+			(end -1.5 -1.25)
+			(stroke
+				(width 0.05)
+				(type solid)
+			)
+			(layer "F.CrtYd")
+		)
+		(fp_line
+			(start -1.5 -1.25)
+			(end -1.5 -1.5)
+			(stroke
+				(width 0.05)
+				(type solid)
+			)
+			(layer "F.CrtYd")
+		)
+		(fp_line
+			(start -1.5 -1.5)
+			(end -1.25 -1.5)
+			(stroke
+				(width 0.05)
+				(type solid)
+			)
+			(layer "F.CrtYd")
+		)
+		(fp_line
+			(start 6.25 5.25)
+			(end 0.25 5.25)
 			(stroke
 				(width 0.1)
@@
 		)
 		(fp_line
-			(start 0.25 5.25)
+			(start 6.25 -0.75)
 			(end 6.25 5.25)
 			(stroke
@@
 		)
 		(fp_line
-			(start 0.25 -0.75)
+			(start 3.25 -0.75)
 			(end 6.25 -0.75)
 			(stroke
@@
 		)
 		(fp_line
+			(start 0.25 5.25)
+			(end 0.25 -0.75)
+			(stroke
+				(width 0.1)
+				(type solid)
+			)
+			(layer "F.Fab")
+		)
+		(fp_line
 			(start 0.25 -0.75)
-			(end 0.25 5.25)
+			(end 3.25 -0.75)
 			(stroke
 				(width 0.1)
@@
 			(layer "F.Fab")
 		)
-		(pad "1" thru_hole rect
-			(at 0 0 180)
-			(size 1.7 1.7)
-			(drill 1)
+		(fp_circle
+			(center 3.25 2.25)
+			(end 1.25 2.5)
+			(stroke
+				(width 0.1)
+				(type solid)
+			)
+			(fill none)
+			(layer "F.Fab")
+		)
+		(fp_text user "${REFERENCE}"
+			(at 3.25 2.25 180)
+			(layer "F.Fab")
+			(effects
+				(font
+					(size 1 1)
+					(thickness 0.15)
+				)
+			)
+		)
+		(pad "1" thru_hole circle
+			(at 0 0 270)
+			(size 2 2)
+			(drill 1.1)
 			(layers "*.Cu" "*.Mask")
 			(remove_unused_layers no)
@@
 		)
 		(pad "1" thru_hole circle
-			(at 6.5 0 180)
-			(size 1.7 1.7)
-			(drill 1)
+			(at 6.5 0 270)
+			(size 2 2)
+			(drill 1.1)
 			(layers "*.Cu" "*.Mask")
 			(remove_unused_layers no)
@@
 		)
 		(pad "2" thru_hole circle
-			(at 0 4.5 180)
-			(size 1.7 1.7)
-			(drill 1)
+			(at 0 4.5 270)
+			(size 2 2)
+			(drill 1.1)
 			(layers "*.Cu" "*.Mask")
 			(remove_unused_layers no)
@@
 		)
 		(pad "2" thru_hole circle
-			(at 6.5 4.5 180)
-			(size 1.7 1.7)
-			(drill 1)
+			(at 6.5 4.5 270)
+			(size 2 2)
+			(drill 1.1)
 			(layers "*.Cu" "*.Mask")
 			(remove_unused_layers no)
@@
 			(pintype "passive")
 		)
-		(model "${KICAD8_3DMODEL_DIR}/Button_Switch_THT.3dshapes/SW_TH_Tactile_Omron_B3F-10xx.wrl"
+		(model "${KICAD8_3DMODEL_DIR}/Button_Switch_THT.3dshapes/SW_PUSH_6mm_H5mm.wrl"
 			(offset
 				(xyz 0 0 0)
@@
 		(tags "Resistor Axial_DIN0204 series Axial Horizontal pin pitch 7.62mm 0.167W length 3.6mm diameter 1.6mm")
 		(property "Reference" "R2"
-			(at 3.81 0 360)
+			(at 3.81 0 0)
 			(layer "F.SilkS")
 			(effects
@@
 		)
 		(property "Value" "1k"
-			(at 3.81 1.92 360)
+			(at 3.81 1.92 0)
 			(layer "F.Fab")
 			(hide yes)
@@
 		)
 		(property "Value" "ICSP"
-			(at 1.15 7.65 0)
+			(at 2.72 7.73 0)
 			(layer "F.SilkS")
 			(effects
@@
 	)
 	(gr_text "+ -"
-		(at 127.39 73.27 180)
+		(at 126.29 73.32 180)
 		(layer "F.SilkS")
 		(effects
