File: Schematic/TH/v2_Beta/Ram_Tester.kicad_pcb (KiCad board)
At the start: 2 copper layers, 63.3 x 57.2 mm, 43 parts, among them J1 Conn_01x02_Pin, J2 ICSP, Q1 2N7000, Q2 2N7000, SW1 SW_DIP_x03, SW2 SW_Push, U1 ATmega328-P, U2 RAM / ZIF, U3 ZIP Socket, Y1 Crystal

Commit message: Add files via upload
Parts:
- Y1: footprint Crystal:Crystal_HC49-U_Vertical -> Crystal:Crystal_HC49-4H_Vertical
Other:
- board text added: "github.com/tops4u/Ram-Tester A.Hoffmann ©2025 License: GPL v3.0"
- board text removed: "github.com/tops4u/Ram-Tester A.Hoffmann ©2024 License: GPL v3.0"
Changed lines of the file:
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@@
 		(sheetname "Root")
 		(sheetfile "Ram_Tester.kicad_sch")
-		(attr through_hole)
+		(attr through_hole dnp)
 		(fp_line
 			(start -1.33 -1.33)
@@
 		(tags "Fuse TE5 Littelfuse/Wickmann No. 460 No560 ")
 		(property "Reference" "F1"
-			(at 2.54 0 270)
+			(at 2.54 0 -90)
 			(layer "F.SilkS")
 			(effects
@@
 		)
 	)
-	(footprint "Crystal:Crystal_HC49-U_Vertical"
+	(footprint "Crystal:Crystal_HC49-4H_Vertical"
 		(layer "F.Cu")
 		(at 100 89.37 -90)
-		(descr "Crystal THT HC-49/U http://5hertz.com/pdfs/04404_D.pdf")
-		(tags "THT crystalHC-49/U")
+		(descr "Crystal THT HC-49-4H http://5hertz.com/pdfs/04404_D.pdf")
+		(tags "THT crystalHC-49-4H")
 		(property "Reference" "Y1"
-			(at 9.2 -2.1 0)
+			(at 2.44 -3.525 -90)
 			(layer "F.SilkS")
 			(effects
@@
 		)
 		(property "Value" "Crystal"
-			(at 2.44 3.525 90)
+			(at 2.44 3.525 -90)
 			(layer "F.Fab")
-			(hide yes)
 			(effects
 				(font
@@
 			)
 		)
-		(property "Footprint" "Crystal:Crystal_HC49-U_Vertical"
+		(property "Footprint" "Crystal:Crystal_HC49-4H_Vertical"
 			(at 0 0 -90)
 			(unlocked yes)
@@
 				(font
 					(size 1.27 1.27)
-					(thickness 0.15)
 				)
 			)
@@
 				(font
 					(size 1.27 1.27)
-					(thickness 0.15)
 				)
 			)
@@
 				(font
 					(size 1.27 1.27)
-					(thickness 0.15)
 				)
 			)
@@
 		(attr through_hole)
 		(fp_line
-			(start -0.685 2.525)
-			(end 5.565 2.525)
+			(start -0.76 2.525)
+			(end 5.64 2.525)
 			(stroke
 				(width 0.12)
@@
 		)
 		(fp_line
-			(start -0.685 -2.525)
-			(end 5.565 -2.525)
+			(start -0.76 -2.525)
+			(end 5.64 -2.525)
 			(stroke
 				(width 0.12)
@@
 		)
 		(fp_arc
-			(start -0.685 2.525)
-			(mid -3.21 0)
-			(end -0.685 -2.525)
+			(start -0.76 2.525)
+			(mid -3.285 0)
+			(end -0.76 -2.525)
 			(stroke
 				(width 0.12)
@@
 		)
 		(fp_arc
-			(start 5.565 -2.525)
-			(mid 8.09 0)
-			(end 5.565 2.525)
+			(start 5.64 -2.525)
+			(mid 8.165 0)
+			(end 5.64 2.525)
 			(stroke
 				(width 0.12)
@@
 		)
 		(fp_line
-			(start -3.5 2.8)
-			(end 8.4 2.8)
+			(start -3.6 2.8)
+			(end 8.5 2.8)
 			(stroke
 				(width 0.05)
@@
 		)
 		(fp_line
-			(start 8.4 2.8)
-			(end 8.4 -2.8)
+			(start 8.5 2.8)
+			(end 8.5 -2.8)
 			(stroke
 				(width 0.05)
@@
 		)
 		(fp_line
-			(start -3.5 -2.8)
-			(end -3.5 2.8)
+			(start -3.6 -2.8)
+			(end -3.6 2.8)
 			(stroke
 				(width 0.05)
@@
 		)
 		(fp_line
-			(start 8.4 -2.8)
-			(end -3.5 -2.8)
+			(start 8.5 -2.8)
+			(end -3.6 -2.8)
 			(stroke
 				(width 0.05)
@@
 		)
 		(fp_line
-			(start -0.685 2.325)
-			(end 5.565 2.325)
+			(start -0.76 2.325)
+			(end 5.64 2.325)
 			(stroke
 				(width 0.1)
@@
 		)
 		(fp_line
-			(start -0.685 -2.325)
-			(end 5.565 -2.325)
+			(start -0.76 -2.325)
+			(end 5.64 -2.325)
 			(stroke
 				(width 0.1)
@@
 		)
 		(fp_arc
-			(start -0.685 2.325)
-			(mid -3.01 0)
-			(end -0.685 -2.325)
+			(start -0.76 2.325)
+			(mid -3.085 0)
+			(end -0.76 -2.325)
 			(stroke
 				(width 0.1)
@@
 		)
 		(fp_arc
-			(start 5.565 -2.325)
-			(mid 7.89 0)
-			(end 5.565 2.325)
+			(start 5.64 -2.325)
+			(mid 7.965 0)
+			(end 5.64 2.325)
 			(stroke
 				(width 0.1)
@@
 			(layer "F.Fab")
 		)
+		(fp_text user "${REFERENCE}"
+			(at 2.44 0 -90)
+			(layer "F.Fab")
+			(effects
+				(font
+					(size 1 1)
+					(thickness 0.15)
+				)
+			)
+		)
 		(pad "1" thru_hole circle
 			(at 0 0 270)
@@
 			(pintype "passive")
 		)
-		(model "${KICAD8_3DMODEL_DIR}/Crystal.3dshapes/Crystal_HC49-U_Vertical.wrl"
+		(model "${KICAD8_3DMODEL_DIR}/Crystal.3dshapes/Crystal_HC49-4H_Vertical.wrl"
 			(offset
 				(xyz 0 0 0)
@@
 		)
 	)
-	(gr_text "github.com/tops4u/Ram-Tester\nA.Hoffmann ©2024\nLicense: GPL v3.0"
+	(gr_text "github.com/tops4u/Ram-Tester\nA.Hoffmann ©2025\nLicense: GPL v3.0"
 		(at 154.1 71.3 0)
 		(layer "F.SilkS")
 		(effects
 			(font
-				(size 1.4 1.1)
+				(size 1.4 1)
 				(thickness 0.2)
 				(bold yes)
