File: Schematic/SMD/Ram_Tester.kicad_sch (KiCad schematic)
At the start: 34 parts, among them J1 Conn_01x04_Pin, J2 ICSP, J3 USB_C_Receptacle_PowerOnly_6P, Q1 IRLML6402, Q2 IRLML6402, SW1 SW_DIP_x03, SW2 SW_Push, U1 ATmega328-P, U2 RAM / ZIF, U3 ZIP Socket, U4 DIP Socket, Y1 Crystal

Commit message: v1.1 of Board
Parts:
- removed U4: DIP Socket, Package_DIP:DIP-20_W7.62mm, symbol Memory_RAM:514256-DIP
- F1: value Fuse -> 0.5A
- Q1, Q2: value IRLML6402 -> BSS138; symbol Transistor_FET:IRLML6402 -> Transistor_FET:BSS138
- R1: value 100 -> 150
- R6: value 150 -> 330
- Y1: value Crystal -> 16MHZ
Connections:
- net 5V2 is gone; now on an unnamed net: C4.2, U3.15 (Vcc)
- net GND2 is gone; now on net GND: C4.1, U3.5 (Vss)
- net 5V: now also D1.1 (A1), D1.2 (A2); no longer Q1.3 (D), Q2.3 (D)
- net GND: now also Q1.2 (S), Q2.2 (S); no longer D1.3 (K1), D1.4 (K2)
- net at RN4.1 (R1.1), U2.19 (I/O4): now also U3.4 (I/O4)
- net at RN4.2 (R2.1), U2.18 (I/O3): now also U3.3 (I/O3)
- net at RN4.3 (R3.1), U2.2 (I/O2): now also U3.7 (I/O2)
- net at RN4.4 (R4.1), U2.1 (I/O1): now also U3.6 (I/O1)
- net at U3.16 (A4): now also RN2.4 (R4.1), U2.11 (A4)
- net at U3.17 (A5): now also RN2.3 (R3.1), U2.12 (A5)
- net at U3.18 (A6): now also RN2.2 (R2.1), U2.13 (A6)
- net at U3.19 (A7): now also RN2.1 (R1.1), U2.14 (A7)
- net at U3.20 (A8): now also R7.2, U2.15 (A8)
- net at U3.1 (OE): now also RN1.2 (R2.1), U2.16 (OE)
- net at U3.2 (CAS): now also RN1.4 (R4.1), U2.17 (CAS)
- net at U3.8 (WE): now also J2.4 (Pin_4), R4.2, RN1.1 (R1.1), RN3.4 (R4.1), SW1.5, U2.3 (WE), U2.9 (A3), U3.14 (A3)
- net at U3.9 (RAS): now also RN1.3 (R3.1), U2.4 (RAS)
- net at U3.10 (N/C): now also R8.2, U2.5 (N/C)
- net at U3.11 (A0): now also RN3.1 (R1.1), U2.6 (A0)
- net at U3.12 (A1): now also RN3.2 (R2.1), U2.7 (A1)
- net at U3.13 (A2): now also R5.2, RN3.3 (R3.1), SW1.4, U2.8 (A2)
- net at R1.1: now also D1.4 (K2); no longer D1.1 (A1)
- net at R1.2: now also Q1.3 (D); no longer Q1.2 (S)
- net at R6.1: now also Q2.3 (D); no longer Q2.2 (S)
- net at R6.2: now also D1.3 (K1); no longer D1.2 (A2)
Other:
- title: (none) -> Ram Tester SMD Version
- moved on the sheet: C4, C7, D1, J1, Q1, Q2, R1, R3, R4, R5, R6, R8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

Commit message: V1.0 fixed
Parts:
- C1, C4, C7: footprint Capacitor_SMD:C_0805_2012Metric -> Capacitor_SMD:C_0603_1608Metric_Pad1.08x0.95mm_HandSolder
- D1: footprint LED_SMD:LED_RGB_Wuerth_150080M153000 -> LED_SMD:LED_SMD_RG_AKAK
Connections:
- net 5V: now also U1.22 (ADC7)
- net GND: no longer U1.22 (ADC7)
- net at R4.2, RN3.4 (R4.1), SW1.5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: no longer J2.4 (Pin_4), RN1.1 (R1.1), U2.3 (WE), U3.8 (WE)
- net at J1.4 (Pin_4), J2.1 (Pin_1), R7.1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: now also Q2.1 (G); no longer Q1.1 (G)
- net at J1.3 (Pin_3), J2.3 (Pin_3), U1.17 (PB5): now also Q1.1 (G); no longer Q2.1 (G)
- net at RN1.8 (R1.2), U1.15 (PB3): now also J2.4 (Pin_4)
- new net: RN1.1 (R1.1), U2.3 (WE), U3.8 (WE)

Commit message: v2.1 Update
Minor Value changes
Parts:
- D1: value LED_Dual_AAKK -> VS 3JD8
- J3: value USB_C_Receptacle_PowerOnly_6P -> KUSBX-SMT-CS-6-BTR
- R1: value 150 -> 150R
- R6: value 330 -> 470R
- R7, R8, RN1, RN2, RN3, RN4: value 47 -> 47R
Changed lines of the file:
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@@
 			)
 		)
-		(property "Value" "47"
+		(property "Value" "47R"
 			(at 205.74 78.7399 0)
 			(effects
@@
 		)
 		(instances
-			(project ""
+			(project "Ram_Tester"
 				(path "/9a90cd34-b6db-44ec-969f-9bfdcecefc17"
 					(reference "U3")
@@
 			)
 		)
-		(property "Value" "47"
+		(property "Value" "47R"
 			(at 111.76 110.744 90)
 			(effects
@@
 		)
 		(instances
-			(project ""
+			(project "Ram_Tester"
 				(path "/9a90cd34-b6db-44ec-969f-9bfdcecefc17"
 					(reference "Y1")
@@
 			)
 		)
-		(property "Value" "47"
+		(property "Value" "47R"
 			(at 188.214 78.74 90)
 			(effects
@@
 			)
 		)
-		(property "Value" "150"
+		(property "Value" "150R"
 			(at 149.86 179.578 90)
 			(effects
@@
 		)
 		(instances
-			(project ""
+			(project "Ram_Tester"
 				(path "/9a90cd34-b6db-44ec-969f-9bfdcecefc17"
 					(reference "F1")
@@
 			)
 		)
-		(property "Value" "330"
+		(property "Value" "470R"
 			(at 132.08 179.578 90)
 			(effects
@@
 		)
 		(instances
-			(project ""
+			(project "Ram_Tester"
 				(path "/9a90cd34-b6db-44ec-969f-9bfdcecefc17"
 					(reference "C3")
@@
 			)
 		)
-		(property "Value" "47"
+		(property "Value" "47R"
 			(at 133.35 63.5 90)
 			(effects
@@
 		)
 		(instances
-			(project ""
+			(project "Ram_Tester"
 				(path "/9a90cd34-b6db-44ec-969f-9bfdcecefc17"
 					(reference "R7")
@@
 		)
 		(instances
-			(project ""
+			(project "Ram_Tester"
 				(path "/9a90cd34-b6db-44ec-969f-9bfdcecefc17"
 					(reference "J2")
@@
 		)
 		(instances
-			(project ""
+			(project "Ram_Tester"
 				(path "/9a90cd34-b6db-44ec-969f-9bfdcecefc17"
 					(reference "SW1")
@@
 		)
 		(instances
-			(project ""
+			(project "Ram_Tester"
 				(path "/9a90cd34-b6db-44ec-969f-9bfdcecefc17"
 					(reference "J1")
@@
 		)
 		(instances
-			(project ""
+			(project "Ram_Tester"
 				(path "/9a90cd34-b6db-44ec-969f-9bfdcecefc17"
 					(reference "U2")
@@
 		)
 		(instances
-			(project ""
+			(project "Ram_Tester"
 				(path "/9a90cd34-b6db-44ec-969f-9bfdcecefc17"
 					(reference "R9")
@@
 			)
 		)
-		(property "Value" "USB_C_Receptacle_PowerOnly_6P"
+		(property "Value" "KUSBX-SMT-CS-6-BTR"
 			(at 29.21 52.07 0)
 			(effects
@@
 		)
 		(instances
-			(project ""
+			(project "Ram_Tester"
 				(path "/9a90cd34-b6db-44ec-969f-9bfdcecefc17"
 					(reference "J3")
@@
 			)
 		)
-		(property "Value" "LED_Dual_AAKK"
+		(property "Value" "VS 3JD8"
 			(at 92.583 176.53 0)
 			(effects
@@
 		)
 		(instances
-			(project ""
+			(project "Ram_Tester"
 				(path "/9a90cd34-b6db-44ec-969f-9bfdcecefc17"
 					(reference "D1")
@@
 		)
 		(instances
-			(project ""
+			(project "Ram_Tester"
 				(path "/9a90cd34-b6db-44ec-969f-9bfdcecefc17"
 					(reference "Q1")
@@
 		)
 		(instances
-			(project ""
+			(project "Ram_Tester"
 				(path "/9a90cd34-b6db-44ec-969f-9bfdcecefc17"
 					(reference "C5")
@@
 		)
 		(instances
-			(project ""
+			(project "Ram_Tester"
 				(path "/9a90cd34-b6db-44ec-969f-9bfdcecefc17"
 					(reference "C2")
@@
 			)
 		)
-		(property "Value" "47"
+		(property "Value" "47R"
 			(at 114.046 133.35 90)
 			(effects
@@
 		)
 		(instances
-			(project ""
+			(project "Ram_Tester"
 				(path "/9a90cd34-b6db-44ec-969f-9bfdcecefc17"
 					(reference "SW2")
@@
 			)
 		)
-		(property "Value" "47"
+		(property "Value" "47R"
 			(at 118.11 66.04 90)
 			(effects
@@
 		)
 		(instances
-			(project ""
+			(project "Ram_Tester"
 				(path "/9a90cd34-b6db-44ec-969f-9bfdcecefc17"
 					(reference "RN1")
@@
 		)
 		(instances
-			(project ""
+			(project "Ram_Tester"
 				(path "/9a90cd34-b6db-44ec-969f-9bfdcecefc17"
 					(reference "U1")
@@
 		)
 		(instances
-			(project ""
+			(project "Ram_Tester"
 				(path "/9a90cd34-b6db-44ec-969f-9bfdcecefc17"
 					(reference "C1")
