File: Schematic/SMD/Ram_Tester.kicad_pcb (KiCad board)
At the start: 2 copper layers, 39.8 x 59.4 mm, 35 parts, among them J1 Conn_01x04_Pin, J2 ICSP, J3 6Pin SMD USB-C, Q1 BSS138, Q2 BSS138, SW1 SW_DIP_x03, SW2 SW_Push, U1 ATmega328-P, U2 RAM / ZIF, U3 ZIP Socket, Y1 16MHZ

Commit message: Completed Design files
Parts:
- moved R1 1.00 mm to (137.0, 66.5)
- moved R6 1.00 mm to (137.0, 68.5)
- moved Q1 0.11 mm to (131.4, 66.5)
Routing:
- net /GND: track 206.2 -> 107.9 mm, vias 63 -> 70
- net MISO: track 77.4 -> 72.2 mm
- net SCK: track 46.1 -> 43.4 mm
- net MOSI: track 33.8 -> 35.5 mm
- net Net-(RN1-R2.1): track 80.9 -> 79.7 mm
- net /5V: track 121.8 -> 122.9 mm, vias 3 -> 5
- net Net-(RN4-R2.1): track 74.5 -> 75.5 mm
